File: comparator/comparator.kicad_pcb (KiCad board)
At the start: 2 copper layers, 40.3 x 110 mm, 5 parts

Commit message: KiCad changes
Parts:
- added C3: 220n, Eurorack:Capacitor Small Non-Polarised, F.Cu at (45.5, 70.0)
- added C4: 100n, Eurorack:Capacitor Small Non-Polarised, F.Cu at (43.0, 75.0)
- added CONN1: Conn_01x08_Male, Connector_PinHeader_2.54mm:PinHeader_2x04_P2.54mm_Vertical, B.Cu at (17.5, 33.3)
- added CONN2: Conn_01x08_Female, Connector_PinSocket_2.54mm:PinSocket_2x04_P2.54mm_Vertical, F.Cu at (48.5, 33.3)
- added CONN3: Conn_01x08_Male, Connector_PinHeader_2.54mm:PinHeader_2x04_P2.54mm_Vertical, B.Cu at (17.5, 52.0)
- added CONN4: Conn_01x08_Female, Connector_PinSocket_2.54mm:PinSocket_2x04_P2.54mm_Vertical, F.Cu at (48.8, 52.0)
- added D3: DIODE, Eurorack:Schottky Diode, F.Cu at (33.2, 41.0)
- added D4: DIODE, Eurorack:Schottky Diode, F.Cu at (37.0, 41.0)
- added IC1: LM2904, Eurorack:DIP-8 IC Socket, F.Cu at (45.0, 40.8)
- added J1: Comparator 2 B, Eurorack:Thonkiconn Mono Jack, F.Cu at (5.00, 83.0)
- added J2: Comparator 1 B, Eurorack:Thonkiconn Mono Jack, F.Cu at (5.00, 22.0)
- added J3: Comparator 2 A, Eurorack:Thonkiconn Mono Jack, F.Cu at (5.00, 69.0)
- added J4: Comparator 1 A, Eurorack:Thonkiconn Mono Jack, F.Cu at (5.00, 8.00)
- added J5: Comparator 2 Out, Eurorack:Thonkiconn Mono Jack, F.Cu at (15.0, 69.0)
- added J6: Comparator 1 Out, Eurorack:Thonkiconn Mono Jack, F.Cu at (15.0, 8.00)
- added LED1: Comparator 1 LED, Eurorack:LED 3mm, F.Cu at (15.0, 21.7)
- added LED2: Comparator 2 LED, Eurorack:LED 3mm, F.Cu at (15.0, 83.0)
- added P1: Comparator 1 Attenuator, Eurorack:Potentiometer 9mm Vertical Linear, F.Cu at (10.0, 47.5)
- added P2: Comparator 1 Attenuator, Eurorack:Potentiometer 9mm Vertical Linear, F.Cu at (10.0, 108.5)
- added Q1: 2N3904, Package_TO_SOT_THT:TO-92_Inline, F.Cu at (48.1, 84.7)
- added Q2: 2N3904, Package_TO_SOT_THT:TO-92_Inline, F.Cu at (43.2, 84.8)
- added R1: 4.7K, Eurorack:Resistor 0.25W Through-Hole Short, F.Cu at (36.2, 68.5)
- added R2: 4.7K, Eurorack:Resistor 0.25W Through-Hole Short, F.Cu at (36.2, 87.8)
- added R3: 100K, Eurorack:Resistor 0.25W Through-Hole Short, F.Cu at (36.2, 71.2)
- added R4: 1K, Eurorack:Resistor 0.25W Through-Hole Short, F.Cu at (36.2, 82.2)
- added R5: 100K, Eurorack:Resistor 0.25W Through-Hole Short, F.Cu at (36.2, 85.0)
- added R6: 100K, Eurorack:Resistor 0.25W Through-Hole Short, F.Cu at (36.2, 76.8)
- added R7: 100K, Eurorack:Resistor 0.25W Through-Hole Short, F.Cu at (36.2, 79.5)
- added R8: 1K, Eurorack:Resistor 0.25W Through-Hole Short, F.Cu at (36.2, 74.0)
- added U1: L7805, Package_TO_SOT_THT:TO-92, F.Cu at (48.8, 64.2)
- EuroPower1: footprint Eurorack:Eurorack Power Header -> Eurorack:Eurorack Power Header Unlabeled; moved to B.Cu
- moved EuroPower1 92.4 mm to (10.0, 94.2), turned to 180 degrees
- moved C1 55.8 mm to (35.7, 53.8), turned to 180 degrees
- moved C2 55.1 mm to (41.8, 53.8), turned to 180 degrees
- moved D1 40.3 mm to (37.0, 30.2), turned to -90 degrees
- moved D2 32.8 mm to (33.2, 30.1), turned to -90 degrees
Connections:
- C1 pad 1: +12V -> /12V B
- C1 pad 2: Earth -> /GND B
- C2 pad 1: Earth -> /GND B
- C2 pad 2: -12V -> /-12V B
- D1 pad 1: Net-(D1-Pad1) -> Net-(CONN4-Pad5)
- D1 pad 2: +12V -> /12V B
- D2 pad 1: -12V -> /-12V B
- EuroPower1 pad 1: Net-(D2-Pad2) -> -12V
- EuroPower1 pad 10: Net-(D1-Pad1) -> +12V
- EuroPower1 pad 2: Net-(D2-Pad2) -> -12V
- EuroPower1 pad 9: Net-(D1-Pad1) -> +12V
Routing:
- net (no net): vias 0 -> 2
Other:
- board size 40.3 x 110 mm -> 51 x 110 mm

Commit message: KiCad changes
Parts:
- D1, D2: footprint Diode_THT:D_DO-41_SOD81_P7.62mm_Horizontal -> Diode_THT:D_A-405_P7.62mm_Horizontal
- turned R1 to 180 degrees
Routing:
- net Earth: track 0.00 -> 177.5 mm, vias 0 -> 3
- net /GND B: track 0.00 -> 107.2 mm, vias 0 -> 3
- net +12V: track 0.00 -> 104.9 mm, vias 0 -> 3
- net Net-(J2-Pad3): track 0.00 -> 90.6 mm, vias 0 -> 1
- net /COM1B A: track 0.00 -> 88.1 mm, vias 0 -> 2
- net -12V: track 0.00 -> 81.0 mm, vias 0 -> 3
- net /COM1LED B: track 0.00 -> 70.5 mm, vias 0 -> 2
- net /12V B: track 0.00 -> 70.1 mm, vias 0 -> 5
- net Net-(D4-Pad1): track 0.00 -> 67.2 mm, vias 0 -> 3
- net Net-(IC1-Pad1): track 0.00 -> 59.6 mm, vias 0 -> 2
- net /COM1OUT B: track 0.00 -> 59.3 mm, vias 0 -> 5
- net Net-(D4-Pad2): track 0.00 -> 54.1 mm, vias 0 -> 2
- net Net-(J1-Pad3): track 0.00 -> 53.1 mm, vias 0 -> 1
- net Net-(D3-Pad2): track 0.00 -> 49.2 mm, vias 0 -> 1
- net Net-(D3-Pad1): track 0.00 -> 49.0 mm
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Other:
- outline, holes or cut-outs redrawn
- board text added: "RED STRIPE"
- board text added: "comparator www.allensynthesis.co.uk CERN OHL-S v2 Designed in Loughborough, UK 01/05/2022"
