File: comparator/comparator.kicad_sch (KiCad schematic)
At the start: 27 parts, among them IC1 LM2904, IC2 LM2904, J1 Comparator 2 B, J2 Comparator 1 B, J3 Comparator 2 A, J4 Comparator 1 A, J5 Comparator 2 Out, J6 Comparator 1 Out, U1 L7805

Commit message: KiCad changes
Parts:
- removed C5, C6, C7: 100n, symbol Device:C
- removed D3: Comparator 2 LED, symbol Device:LED
- removed IC2: LM2904, symbol Amplifier_Operational:LM2904
- removed P?: Comparator 2 Attenuator, symbol Eurorack:Potentiometer_9mm_Vertical_Linear
- added CONN1, CONN3: Conn_01x08_Male, Connector_PinHeader_2.54mm:PinHeader_2x04_P2.54mm_Vertical, symbol Connector:Conn_01x08_Male
- added CONN2, CONN4: Conn_01x08_Female, Connector_PinSocket_2.54mm:PinSocket_2x04_P2.54mm_Vertical, symbol Connector:Conn_01x08_Female
- added D3, D4: DIODE, Eurorack:Schottky Diode, symbol Simulation_SPICE:DIODE
- added LED2: Comparator 2 LED, Eurorack:LED 3mm, symbol Device:LED
- added P1: Comparator 1 Attenuator, Eurorack:Potentiometer 9mm Vertical Linear, symbol Eurorack:Potentiometer_9mm_Vertical_Linear
- added Q1, Q2: 2N3904, Package_TO_SOT_THT:TO-92_Inline, symbol Transistor_BJT:2N3904
- added R5, R6, R7: 100K, Eurorack:Resistor 0.25W Through-Hole Short, symbol Device:R
- added R8: 1K, Eurorack:Resistor 0.25W Through-Hole Short, symbol Device:R
- C3, C4: footprint (none) -> Eurorack:Capacitor Small Non-Polarised
- EuroPower1: footprint Eurorack:Eurorack Power Header -> Eurorack:Eurorack Power Header Unlabeled
- IC1: footprint (none) -> Eurorack:DIP-8 IC Socket
- J1, J2, J3, J4, J5, J6: footprint (none) -> Eurorack:Thonkiconn Mono Jack
- LED1: renamed from D4; footprint (none) -> Eurorack:LED 3mm
- P2: renamed from P?; footprint (none) -> Eurorack:Potentiometer 9mm Vertical Linear
- R1, R2, R4: footprint (none) -> Eurorack:Resistor 0.25W Through-Hole Short
- R3: value 1K -> 100K; footprint (none) -> Eurorack:Resistor 0.25W Through-Hole Short
- U1: footprint (none) -> Package_TO_SOT_THT:TO-92
Connections:
- net +12V: now also EuroPower1.10 (Pin_10), EuroPower1.9 (Pin_9), CONN1.5 (Pin_5), CONN3.5 (Pin_5); no longer C1.1, C3.1, D1.2 (K), IC1.8 (V+), U1.1 (IN)
- net +5V: now also Q1.3 (C), Q2.3 (C)
- net -12V: now also EuroPower1.1 (Pin_1), EuroPower1.2 (Pin_2), CONN1.8 (Pin_8), CONN3.8 (Pin_8); no longer C2.2, D2.1 (A), IC1.4 (V-)
- net Earth: now also CONN1.6 (Pin_6), CONN1.7 (Pin_7), CONN3.6 (Pin_6), CONN3.7 (Pin_7), LED2.1 (K), P1.1; no longer C1.2, C2.1, C3.2, C4.2, U1.2 (GND)
- net at IC1.1, R2.1: now also R5.2
- net COM1LED A: now reaches LED1.2 (A)
- net COM1LED A: now also CONN1.4 (Pin_4); no longer R2.2
- net at IC1.7, R1.1: now also R3.2
- net COM2LED B: now reaches R1.2
- net COM2LED B: now also CONN4.4 (Pin_4)
- net at J1.3 (T): now also P1.3
- net at R3.1: now also D4.1 (A), Q1.2 (B)
- net COM2OUT A: now reaches J5.3 (T)
- net COM2OUT A: now also CONN3.3 (Pin_3); no longer R3.2
- net COM2A A: now reaches J3.3 (T)
- net COM2A A: now also CONN3.1 (Pin_1); no longer IC1.5 (+)
- net at R4.1: now also D3.2 (K), Q2.1 (E), R7.2
- net COM2B B: now reaches IC1.6 (-)
- net COM2B B: now also CONN4.2 (Pin_2)
- net COM1B A: now reaches P2.2
- net COM1B A: now also CONN1.2 (Pin_2); no longer IC1.2 (-)
- net COM1A A: now reaches J4.3 (T)
- net COM1A A: now also CONN1.1 (Pin_1); no longer IC1.3 (+)
- net COM1OUT A: now reaches J6.3 (T)
- net COM1OUT A: now also CONN1.3 (Pin_3); no longer R4.2
- new net: D4.2 (K), Q1.1 (E), R6.2, R8.1
- new net: D3.1 (A), Q2.2 (B), R5.1
- new net: CONN4.8 (Pin_8), D2.2 (K)
- new net: CONN4.5 (Pin_5), D1.1 (A)
- new net -12V B: C2.2, CONN2.8 (Pin_8), D2.1 (A), IC1.4 (V-)
- new net 12V B: C1.1, C3.1, CONN2.5 (Pin_5), D1.2 (K), IC1.8 (V+), U1.1 (IN)
- new net COM1A B: CONN2.1 (Pin_1), IC1.3 (+)
- new net COM1B B: CONN2.2 (Pin_2), IC1.2 (-)
- new net COM1LED B: CONN2.4 (Pin_4), R2.2
- new net COM1OUT B: CONN2.3 (Pin_3), R4.2
- new net COM2A B: CONN4.1 (Pin_1), IC1.5 (+)
- new net COM2B A: CONN3.2 (Pin_2), P1.2
- new net COM2LED A: CONN3.4 (Pin_4), LED2.2 (A)
- new net COM2OUT B: CONN4.3 (Pin_3), R8.2
- new net GND B: C1.2, C2.1, C3.2, C4.2, CONN2.6 (Pin_6), CONN2.7 (Pin_7), CONN4.6 (Pin_6), CONN4.7 (Pin_7), R6.1, R7.1, U1.2 (GND)
Other:
- moved on the sheet: D1, D2, J2, J4, J6, LED1, P2, R2, R4

Commit message: KiCad changes
Parts:
- D1, D2: footprint Diode_THT:D_DO-41_SOD81_P7.62mm_Horizontal -> Diode_THT:D_A-405_P7.62mm_Horizontal
Changed lines of the file:
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@@
     (property "Reference" "D2" (id 0) (at 254.635 162.56 0))
     (property "Value" "DIODE" (id 1) (at 254.635 164.465 0))
-    (property "Footprint" "Diode_THT:D_DO-41_SOD81_P7.62mm_Horizontal" (id 2) (at 254.635 159.385 0)
+    (property "Footprint" "Diode_THT:D_A-405_P7.62mm_Horizontal" (id 2) (at 254.635 159.385 0)
       (effects (font (size 1.27 1.27)) hide)
     )
@@
     (property "Reference" "D1" (id 0) (at 254.635 146.685 0))
     (property "Value" "DIODE" (id 1) (at 254.635 148.59 0))
-    (property "Footprint" "Diode_THT:D_DO-41_SOD81_P7.62mm_Horizontal" (id 2) (at 254.635 151.765 0)
+    (property "Footprint" "Diode_THT:D_A-405_P7.62mm_Horizontal" (id 2) (at 254.635 151.765 0)
       (effects (font (size 1.27 1.27)) hide)
     )
@@
     )
     (path "/a65de6f7-a57d-4433-8d00-2faaf28702a5"
-      (reference "D1") (unit 1) (value "DIODE") (footprint "Diode_THT:D_DO-41_SOD81_P7.62mm_Horizontal")
+      (reference "D1") (unit 1) (value "DIODE") (footprint "Diode_THT:D_A-405_P7.62mm_Horizontal")
     )
     (path "/5b17d47a-a4a2-4ddf-966a-e6b5821094ec"
-      (reference "D2") (unit 1) (value "DIODE") (footprint "Diode_THT:D_DO-41_SOD81_P7.62mm_Horizontal")
+      (reference "D2") (unit 1) (value "DIODE") (footprint "Diode_THT:D_A-405_P7.62mm_Horizontal")
     )
     (path "/bc704d96-cc18-45a3-8762-752ec6ff2845"
